File: MoonHub.kicad_pcb (KiCad board)
At the start: 4 copper layers, 102 x 16.5 mm, 38 parts, among them J1 X1224WRS-04-LPV01, U1 AP22818AKBWT-7, U2 H5VU25U, U3 H5VU25U, U4 CH334U, U5 H5VU25U, Y1 12MHz

Commit message: change ESD
Parts:
- removed the G*** at (29.7, 1.90)
Other:
- board text removed: "a design by"
